Commit message: fix: correct lefT_hip_yaw_joint typo to left_hip_yaw_joint

File: src/holosoma_retargeting/holosoma_retargeting/models/irmv_v3/irmv_v3_21dof.urdf (robot description, URDF)
Before this commit: robot irmv_v3, 22 links, 21 joints
Joints:
- removed joint lefT_hip_yaw_joint
- added joint left_hip_yaw_joint: type revolute, parent left_hip_roll_link, child left_hip_yaw_link, origin xyz=0 0 -0.080622 rpy=0 0 0, axis 0 0 1, limit lower=-1.15 upper=1.15 effort=50 velocity=0
